File: mini-65.kicad_pcb (KiCad board)
At the start: 2 copper layers, 173 parts, among them J1 AVR-ISP-6, SW1 SW_Push, U1 ATmega32U4-AU, Y1 Crystal_GND24_Small

Commit message: Laid out keys on the PCB.
Parts:
- MX_ISO_ENTER1: footprint MX_Alps_Hybrid:MX-ISO -> MX_Only:MXOnly-ISO-ROTATED-ReversedStabilizers-NoLED
- moved SW1 623.1 mm to (-355.7, 102.1)
- moved C2 465.6 mm to (-347.1, 175.3)
- moved C3 465.6 mm to (-347.1, 178.3)
- moved C4 465.6 mm to (-347.1, 181.2)
- moved C5 465.6 mm to (-347.1, 184.2)
- moved C6 465.6 mm to (-347.1, 187.1)
- moved F1 393.7 mm to (-355.9, 156.4)
- moved Y1 393.7 mm to (-356.1, 160.3)
- moved D1 373.4 mm to (-263.6, 64.7)
- moved D11 373.4 mm to (-357.0, 58.1)
- moved D12 373.4 mm to (-377.8, 54.5)
- moved D14 373.4 mm to (-377.8, 58.1)
- moved D16 373.4 mm to (-273.8, 57.5)
- moved D17 373.4 mm to (-273.8, 53.9)
- moved D19 373.4 mm to (-273.8, 50.3)
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- renumbered MX_10 to MX_0, MX_11 to MX_DASH1, MX_12 to MX_EQUALS1

Commit message: Set MCU to the side
Parts:
- moved D64 449.1 mm to (46.2, 64.0)
- moved D1 434.7 mm to (170.9, 74.0)
- moved D16 434.7 mm to (160.8, 66.8)
- moved D17 434.7 mm to (160.8, 63.2)
- moved D19 434.7 mm to (160.8, 59.6)
- moved D26 434.7 mm to (160.8, 70.4)
- moved D10 434.7 mm to (160.5, 74.0)
- moved D11 434.7 mm to (77.6, 67.4)
- moved D12 434.7 mm to (56.8, 63.8)
- moved D13 434.7 mm to (67.2, 63.8)
- moved D14 434.7 mm to (56.8, 67.4)
- moved D15 434.7 mm to (150.4, 63.2)
- moved D2 434.7 mm to (181.6, 66.8)
- moved D20 434.7 mm to (150.4, 70.4)
- moved D21 434.7 mm to (150.4, 66.8)
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
Commit message: Switched around ISO enter and ISO backslash
Parts:
- moved D68 205.7 mm to (235.5, 172.6)
- moved D69 200.3 mm to (256.0, 172.8)
- moved D60 194.6 mm to (258.7, 153.7)
- moved D67 192.8 mm to (212.2, 172.6)
- moved D1 190.6 mm to (-19.1, 89.7), turned to 90 degrees
- moved D16 187.4 mm to (-19.9, 116.5)
- moved D59 185.9 mm to (241.2, 152.1)
- moved D58 183.1 mm to (210.2, 152.4)
- moved D2 183.0 mm to (0.00, 89.7), turned to 90 degrees
- moved D45 180.0 mm to (257.7, 134.0)
- moved D66 172.7 mm to (188.3, 172.2)
- moved D17 168.2 mm to (1.02, 115.6)
- moved D31 167.3 mm to (-23.0, 135.4)
- moved D3 164.7 mm to (19.1, 89.7), turned to 90 degrees
- moved D14 164.2 mm to (218.6, 95.6)
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
Commit message: Rearranged diodes
Parts:
- moved D29 41.3 mm to (247.7, 109.5), turned to 90 degrees
- moved D43 26.8 mm to (207.2, 127.8), turned to 90 degrees
- moved D2 18.3 mm to (-18.3, 89.7)
- moved D3 18.3 mm to (0.79, 89.7)
- moved D1 18.3 mm to (-37.3, 89.7)
- moved D16 14.1 mm to (-31.8, 108.7), turned to 90 degrees
- moved D12 13.5 mm to (172.2, 89.7), turned to 90 degrees
- moved D31 13.4 mm to (-11.9, 127.8), turned to 90 degrees
- moved D67 13.4 mm to (223.8, 165.9), turned to 90 degrees
- moved D69 12.7 mm to (266.7, 165.9), turned to 90 degrees
- moved D5 12.7 mm to (38.9, 89.7), turned to 90 degrees
- moved D49 12.7 mm to (42.9, 146.8), turned to 90 degrees
- moved D13 12.7 mm to (191.3, 89.7), turned to 90 degrees
- moved D62 12.6 mm to (9.53, 165.9), turned to 90 degrees
- moved D64 12.6 mm to (114.3, 165.9), turned to 90 degrees
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Connections:
- MX_ISO_ENTER1 pad 1: COL12 -> COL13
- MX_ISO_ENTER1 pad 2: Net-(D43-Pad2) -> Net-(D29-Pad2)
- MX_ISO_\1 pad 1: COL13 -> COL12
- MX_ISO_\1 pad 2: Net-(D29-Pad2) -> Net-(D43-Pad2)

Commit message: changed location of diodes
Parts:
- moved D43 28.8 mm to (235.7, 131.8)
- moved D46 25.4 mm to (-35.7, 146.8)
- moved D31 24.6 mm to (-36.5, 127.8)
- moved D61 21.4 mm to (-35.7, 165.9)
- moved D2 19.1 mm to (0.79, 89.7)
- moved D30 17.5 mm to (249.2, 108.7)
- moved D11 17.5 mm to (170.7, 89.7)
- moved D12 17.5 mm to (189.7, 89.7)
- moved D13 17.5 mm to (208.8, 89.7)
- moved D22 17.5 mm to (104.8, 108.7)
- moved D23 17.5 mm to (123.8, 108.7)
- moved D24 17.5 mm to (142.9, 108.7)
- moved D25 17.5 mm to (161.9, 108.7)
- moved D26 17.5 mm to (181.0, 108.7)
- moved D27 17.5 mm to (200.0, 108.7)
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
Commit message: Moved around some of the diode locations
Parts:
- removed MX_1.25U_RSHIFT1: MX-NoLED, MX_Alps_Hybrid:MX-1.25U-NoLED
- removed MX_FN_2, MX_TEMP2: MX-NoLED, MX_Alps_Hybrid:MX-1U-NoLED
- MX_'1, MX_,1, MX_.1, MX_/1, MX_0, MX_1, MX_2, MX_3, MX_4, MX_5, MX_6, MX_7, MX_8, MX_9, MX_;1, MX_A1, MX_ARR_D1, MX_ARR_L1, MX_ARR_R1, MX_ARR_U1, MX_B1, MX_BACKSPACE_1u1, MX_BACKSP_EXTRA1, MX_C1, MX_D1, MX_DASH1, MX_DEL1, MX_E1, MX_EQUALS1, MX_ESC1, MX_F1, MX_G1, MX_H1, MX_I1, MX_INS1, MX_ISO_\1, MX_J1, MX_K1, MX_L1, MX_L_BSLASH1, MX_L_WIN1, MX_M1, MX_N1, MX_O1, MX_P1, MX_PrtSc1, MX_Q1, MX_R1, MX_R_WIN1, MX_S1, MX_STEP_CAPS1, MX_T1, MX_TEMP1, MX_U1, MX_V1, MX_W1, MX_X1, MX_Y1, MX_Z1, MX_[1, MX_]1: footprint MX_Alps_Hybrid:MX-1U-NoLED -> MX_Only:MXOnly-1U-NoLED
- MX_1.25U_FN1, MX_1.25U_L_ALT1, MX_1.25U_L_CTRL1, MX_1.25U_L_SHIFT1, MX_1.25U_L_WIN1, MX_1.25U_R_CTRL1, MX_1.25U_R_CTRL2, MX_1.25U_R_FN1: footprint MX_Alps_Hybrid:MX-1.25U-NoLED -> MX_Only:MXOnly-1.25U-NoLED
- MX_1.5U_L_ALT1, MX_1.5U_L_CTRL1, MX_1.5U_R_ALT1, MX_1.5U_R_CTRL1, MX_1.5U_TAB1, MX_1.5U_\1: footprint MX_Alps_Hybrid:MX-1.5U-NoLED -> MX_Only:MXOnly-1.5U-NoLED
- MX_1.75U_CAPSLOCK1, MX_1.75U__RSHIFT1: footprint MX_Alps_Hybrid:MX-1.75U-NoLED -> MX_Only:MXOnly-1.75U-NoLED
- MX_2.25U_ENTER1, MX_2.25U_LSHIFT1: footprint MX_Alps_Hybrid:MX-2.25U-NoLED -> MX_Only:MXOnly-2.25U-NoLED
- MX_2.75U_RSHIFT1: footprint MX_Alps_Hybrid:MX-2.75U-NoLED -> MX_Only:MXOnly-2.75U-NoLED
- MX_2U_BACKSP1: footprint MX_Alps_Hybrid:MX-2U-NoLED -> MX_Only:MXOnly-2U-NoLED
- MX_6.25U_SPACE1: footprint MX_Alps_Hybrid:MX-6.25U-NoLED -> MX_Only:MXOnly-6.25U-NoLED
- MX_7U_SPACE1: footprint MX_Alps_Hybrid:MX-7U-NoLED -> MX_Only:MXOnly-7U-NoLED
- moved D58 31.0 mm to (230.2, 146.8)
- moved D31 23.8 mm to (-12.7, 127.8)
- moved D46 23.1 mm to (-12.7, 148.4)
- moved D16 21.4 mm to (-15.1, 108.7)
- moved D61 21.4 mm to (-14.3, 165.9)
- moved D30 17.5 mm to (266.7, 108.7)
- moved D45 17.5 mm to (266.7, 127.8)
- moved D1 16.7 mm to (-19.8, 89.7)
- moved D43 12.6 mm to (247.7, 127.8)
- moved D29 8.87 mm to (247.7, 108.7)
- moved MX_ARR_L1 4.76 mm to (219.9, 166.7)
- moved MX_ARR_D1 4.76 mm to (238.9, 166.7)
- moved MX_ARR_R1 4.76 mm to (258.0, 166.7)
- moved MX_ARR_U1 4.76 mm to (238.9, 147.6)
- moved D68 3.18 mm to (247.7, 165.9)
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Connections:
- MX_1.25U_FN1 pad 1: COL10 -> COL11
- MX_1.25U_R_CTRL1 pad 1: COL9 -> COL10
- MX_1.5U_R_CTRL1 pad 1: COL10 -> COL11

Commit message: Moved the diodes down a bit
Parts:
- removed D44: 1N4148W, canadian_footprints:D_SOD123_axial-dual
- removed MX_BACKSPACE_1u1, MX_BACKSP_EXTRA1: MX-NoLED, MX_Only:MXOnly-1U-NoLED
- moved D14 25.5 mm to (237.3, 92.1)
- moved D67 24.7 mm to (202.4, 168.3)
- moved D31 23.1 mm to (-35.7, 129.4)
- moved D46 23.0 mm to (-35.7, 149.2)
- moved D61 21.6 mm to (-35.7, 168.3)
- moved D16 20.8 mm to (-35.7, 111.1)
- moved D1 16.1 mm to (-35.7, 92.1)
- moved D52 2.86 mm to (99.2, 149.2)
- moved D49 2.86 mm to (42.1, 149.2)
- moved D41 2.51 mm to (184.9, 130.2)
- moved D43 2.51 mm to (246.9, 130.2)
- moved D34 2.51 mm to (51.6, 130.2)
- moved D35 2.51 mm to (70.6, 130.2)
- moved D36 2.51 mm to (89.7, 130.2)
- moved D38 2.51 mm to (127.8, 130.2)
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Routing:
- net COL12: track 0.00 -> 104.1 mm
- net COL0: track 0.00 -> 100.9 mm
- net COL6: track 0.00 -> 99.0 mm
- net COL13: track 0.00 -> 95.0 mm
- net COL2: track 0.00 -> 91.4 mm
- net COL1: track 0.00 -> 89.4 mm
- net COL11: track 0.00 -> 88.4 mm
- net COL10: track 0.00 -> 88.0 mm
- net COL14: track 0.00 -> 76.2 mm
- net COL9: track 0.00 -> 67.0 mm
- net COL5: track 0.00 -> 67.0 mm
- net COL4: track 0.00 -> 67.0 mm
- net COL8: track 0.00 -> 67.0 mm
- net COL7: track 0.00 -> 67.0 mm
- net COL3: track 0.00 -> 67.0 mm
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Other:
- net class Default: trace_width 0.25 -> 0.254
- net class Power added: clearance 0.2, trace_width 0.381, via_dia 0.8, via_drill 0.4

Commit message: Routed all rows/colums,  started on controller design
Parts:
- C1, C2, C3, C4, C5, C6, C7, J1, R1, R4, SW1, Y1: moved to B.Cu
- moved C2 167.8 mm to (31.0, 190.0), turned to 45 degrees
- moved Y1 159.5 mm to (27.9, 186.9), turned to 315 degrees
- moved C1 152.4 mm to (25.1, 184.2), turned to 225 degrees
- moved SW1 135.1 mm to (69.8, 197.6)
- moved R1 132.0 mm to (13.4, 200.8)
- moved C7 128.3 mm to (13.4, 197.8)
- moved C3 126.8 mm to (8.53, 199.5)
- moved C4 123.8 mm to (8.53, 196.6)
- moved C5 121.0 mm to (8.53, 193.6)
- moved R4 118.5 mm to (13.4, 189.0)
- moved C6 118.5 mm to (8.53, 190.7)
- moved J1 114.5 mm to (27.8, 200.0)
- moved U1 100.7 mm to (31.8, 161.9), turned to 0 degrees
- moved F1 56.8 mm to (-55.6, 97.6), turned to 90 degrees
- moved D12 42.1 mm to (147.6, 90.5)
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Routing:
- net ROW1: track 0.00 -> 303.0 mm
- net ROW3: track 0.00 -> 301.6 mm
- net ROW2: track 0.00 -> 301.6 mm
- net ROW4: track 0.00 -> 301.6 mm
- net ROW0: track 0.00 -> 301.6 mm
- net GND: track 0.00 -> 179.4 mm
- net Net-(R2-Pad1): track 0.00 -> 158.9 mm
- net Net-(R3-Pad1): track 0.00 -> 157.5 mm
- net +5V: track 0.00 -> 154.8 mm
- net Net-(D43-Pad2): track 0.00 -> 30.4 mm
- net Net-(D29-Pad2): track 0.00 -> 27.9 mm
- net Net-(D67-Pad2): track 2.38 -> 21.1 mm
- net Net-(D16-Pad2): track 0.00 -> 16.4 mm
- net Net-(D14-Pad2): track 0.00 -> 16.1 mm
- net D+: track 0.00 -> 14.1 mm
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Other:
- board outline added: 308 x 98.4 mm
