File: _autosave-mini-65.sch (KiCad schematic (older format))
At the start: 170 parts, among them J1 TYPE-C-31-M12_13_EDITED, J2 AVR-ISP-6, SW1 SW_Push, U1 ATmega32U4-AU, U2 USBLC6-2SC6, Y1 Crystal_GND24_Small

Commit message: All col/rows routed, ground screw pads extended
Connections:
- wire segments 325 -> 324
Changed lines of the file:
@@
 Connection ~ 12800 1050
-Wire Wire Line
-	12850 550  13350 550
 Wire Wire Line
 	11300 4350 11900 4350
@@
 Wire Wire Line
 	8550 6350 8550 6400
-Text GLabel 7300 6350 2    50   Input ~ 0
+Text GLabel 3150 2950 2    50   Input ~ 0
 ROW0
-Text GLabel 7300 6250 2    50   Input ~ 0
+Text GLabel 3150 2050 2    50   Input ~ 0
 ROW1
-Text GLabel 7300 6150 2    50   Input ~ 0
+Text GLabel 3150 2850 2    50   Input ~ 0
 ROW2
-Text GLabel 7600 4950 2    50   Input ~ 0
+Text GLabel 3150 2750 2    50   Input ~ 0
 COL14
-Text GLabel 7600 5050 2    50   Input ~ 0
+Text GLabel 3150 3150 2    50   Input ~ 0
 COL13
-Text GLabel 7600 5150 2    50   Input ~ 0
+Text GLabel 3150 3250 2    50   Input ~ 0
 COL12
-Text GLabel 7600 5250 2    50   Input ~ 0
+Text GLabel 3150 1750 2    50   Input ~ 0
 COL11
-Text GLabel 7600 5350 2    50   Input ~ 0
+Text GLabel 3150 1850 2    50   Input ~ 0
 COL10
-Text GLabel 7600 5450 2    50   Input ~ 0
+Text GLabel 3150 1950 2    50   Input ~ 0
 COL9
-Text GLabel 7600 5550 2    50   Input ~ 0
+Text GLabel 3150 2650 2    50   Input ~ 0
 COL8
-Text GLabel 7600 5650 2    50   Input ~ 0
+Text GLabel 3150 2550 2    50   Input ~ 0
 COL7
-Text GLabel 7600 5750 2    50   Input ~ 0
+Text GLabel 3150 2250 2    50   Input ~ 0
 COL6
-Text GLabel 7600 5850 2    50   Input ~ 0
+Text GLabel 3150 3550 2    50   Input ~ 0
 COL5
-Text GLabel 7600 5950 2    50   Input ~ 0
+Text GLabel 3150 3750 2    50   Input ~ 0
 COL4
-Text GLabel 7600 6050 2    50   Input ~ 0
+Text GLabel 3150 3850 2    50   Input ~ 0
 COL3
-Text GLabel 7300 6050 2    50   Input ~ 0
+Text GLabel 3150 3950 2    50   Input ~ 0
 ROW3
-Text GLabel 7600 6350 2    50   Input ~ 0
+Text GLabel 3150 4050 2    50   Input ~ 0
 COL0
-Text GLabel 7600 6250 2    50   Input ~ 0
+Text GLabel 3150 4150 2    50   Input ~ 0
 COL1
-Text GLabel 7600 6150 2    50   Input ~ 0
+Text GLabel 3150 4250 2    50   Input ~ 0
 COL2
-Text GLabel 7300 5950 2    50   Input ~ 0
+Text GLabel 3150 2350 2    50   Input ~ 0
 ROW4
 $EndSCHEMATC
