File: _autosave-mini-65.kicad_pcb (KiCad board)
At the start: 2 copper layers, 303.5 x 94 mm, 170 parts, among them J1 TYPE-C-31-M12_13_EDITED, J2 AVR-ISP-6, SW1 SW_Push, U1 ATmega32U4-AU, U2 USBLC6-2SC6, Y1 Crystal_GND24_Small

Commit message: Tweaked the MX footprints to include plated holes
Parts:
- moved D1 13.2 mm to (-77.8, 87.7), turned to 90 degrees
- moved D31 2.79 mm to (-54.8, 125.8)
- moved D32 2.79 mm to (-28.6, 125.8)
- moved D33 2.79 mm to (-9.53, 125.8)
- moved D34 2.79 mm to (9.53, 125.8)
- moved D35 2.79 mm to (28.6, 125.8)
- moved D36 2.79 mm to (31.8, 125.8)
- moved D37 2.79 mm to (66.7, 125.8)
- moved D38 2.79 mm to (85.7, 125.8)
- moved D39 2.79 mm to (104.8, 125.8)
- moved D40 2.79 mm to (123.8, 125.8)
- moved D41 2.79 mm to (142.9, 125.8)
- moved D42 2.79 mm to (161.9, 125.8)
- moved D43 2.79 mm to (204.8, 125.8)
- moved D44 2.79 mm to (208.0, 125.8)
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Routing:
- net GND: track 943.4 -> 1005.6 mm
- net ROW0: track 558.5 -> 574.0 mm
- net Net-(D1-Pad2): track 17.1 -> 10.5 mm
- net ROW2: track 500.7 -> 505.5 mm
- net ROW1: track 335.6 -> 338.0 mm
- net Net-(D16-Pad2): track 10.5 -> 12.9 mm
- net ROW3: track 354.8 -> 353.2 mm
- net Net-(D14-Pad2): track 16.1 -> 14.9 mm
- net Net-(D12-Pad2): track 6.54 -> 5.41 mm
- net Net-(D15-Pad2): track 11.6 -> 10.5 mm
- net Net-(D7-Pad2): track 6.54 -> 5.41 mm
- net Net-(D2-Pad2): track 6.54 -> 5.41 mm
- net Net-(D9-Pad2): track 6.54 -> 5.41 mm
- net Net-(D8-Pad2): track 6.54 -> 5.41 mm
- net Net-(D6-Pad2): track 6.54 -> 5.41 mm
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
Commit message: Update _autosave-mini-65.kicad_pcb
Parts:
- MX_'1, MX_,1, MX_.1, MX_/1, MX_0, MX_1, MX_2, MX_3, MX_4, MX_5, MX_6, MX_7, MX_8, MX_9, MX_;1, MX_A1, MX_ARR_D1, MX_ARR_L1, MX_ARR_R1, MX_ARR_U1, MX_B1, MX_C1, MX_D1, MX_DASH1, MX_DEL1, MX_E1, MX_EQUALS1, MX_ESC1, MX_F1, MX_FN1, MX_G1, MX_H1, MX_I1, MX_INS1, MX_ISO_\1, MX_J1, MX_K1, MX_L1, MX_L_ALT1, MX_L_BSLASH1, MX_M1, MX_N1, MX_O1, MX_P1, MX_PrtSc1, MX_Q1, MX_R1, MX_R_CTRL1, MX_S1, MX_STEP_CAPS1, MX_T1, MX_TEMP1, MX_U1, MX_V1, MX_W1, MX_X1, MX_Y1, MX_Z1, MX_[1, MX_]1: footprint MX_Only:MXOnly-1U-NoLED -> mini-MX-Tweaks:MXOnly-1U-NoLED_tweak
- MX_1.25U_FN1, MX_1.25U_L_ALT1, MX_1.25U_L_CTRL1, MX_1.25U_L_SHIFT1, MX_1.25U_L_WIN1, MX_1.25U_R_CTRL1: footprint MX_Only:MXOnly-1.25U-NoLED -> mini-MX-Tweaks:MXOnly-1.25U-NoLED_tweak
- MX_1.5U_TAB1, MX_1.5U_\1: footprint MX_Only:MXOnly-1.5U-NoLED -> mini-MX-Tweaks:MXOnly-1.5U-NoLED_tweak
- MX_1.75U_CAPSLOCK1, MX_1.75U__RSHIFT1: footprint MX_Only:MXOnly-1.75U-NoLED -> mini-MX-Tweaks:MXOnly-1.75U-NoLED_tweak
- MX_2.25U_ENTER1, MX_2.25U_LSHIFT1: footprint MX_Only:MXOnly-2.25U-NoLED -> mini-MX-Tweaks:MXOnly-2.25U-NoLED_tweak
- MX_2U_BACKSP1: footprint MX_Only:MXOnly-2U-NoLED -> mini-MX-Tweaks:MXOnly-2U-NoLED_tweak
- MX_6.25U_SPACE1: footprint MX_Only:MXOnly-6.25U-ReversedStabilizers-NoLED -> mini-MX-Tweaks:MXOnly-6.25U-ReversedStabilizers-NoLED_tweak
- MX_ISO_ENTER1: footprint MX_Only:MXOnly-ISO-ROTATED-ReversedStabilizers-NoLED -> mini-MX-Tweaks:MXOnly-ISO-ROTATED-ReversedStabilizers-NoLED_tweak
