File: mini-eLiXiVy.kicad_pcb (KiCad board)
At the start: 2 copper layers, 302.2 x 93.5 mm, 175 parts, among them J1 TYPE-C-31-M12_13_EDITED, J2 AVR-ISP-6, SW1 SW_Push, U1 ATmega32U4-AU, U2 WE-TVS-82400102, Y1 Crystal_GND24_Small

Commit message: rev.1a minor changes
Other:
- board text removed: "JLCJLCJLCJLC"
Changed lines of the file:
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@@
   (general
     (thickness 1.6)
-    (drawings 25)
+    (drawings 24)
     (tracks 1406)
     (zones 0)
@@
       (creategerberjobfile false)
       (excludeedgelayer true)
-      (linewidth 0.100000)
+      (linewidth 0.020000)
       (plotframeref false)
       (viasonmask false)
@@
       (drillshape 0)
       (scaleselection 1)
-      (outputdirectory "Releases/Rev1a/PCB Gerber/"))
+      (outputdirectory "Gerbers/rev.1a"))
   )
   (net 0 "")
@@
     (effects (font (size 1 1) (thickness 0.15)) (justify mirror))
   )
-  (gr_text JLCJLCJLCJLC (at 24.765 105.37825) (layer F.SilkS)
-    (effects (font (size 0.81 0.81) (thickness 0.16)))
-  )
   (gr_text "ANSI\nSHIFT" (at 34.163 85.43925) (layer F.SilkS)
